Commit message: Fixed racecar-description issues

File: cartographer_config/racecar_description/urdf/macros.xacro (robot description, xacro)
@@ -41,5 +41,5 @@
   <origin xyz="0 0 0" rpy="0 0 0" />
   <geometry>
-    <mesh filename="package://racecar_description/meshes/chassis.STL" />
+    <mesh filename="$(find maze_solver)/cartographer_config/racecar_description/meshes/chassis.STL" />
   </geometry>
 </xacro:macro>
@@ -47,5 +47,5 @@
   <origin xyz="0 0 0" rpy="0 0 0" />
   <geometry>
-    <mesh filename="package://racecar_description/meshes/left_rear_wheel.STL" />
+    <mesh filename="$(find maze_solver)/cartographer_config/racecar_description/meshes/left_rear_wheel.STL" />
   </geometry>
 </xacro:macro>
@@ -53,5 +53,5 @@
   <origin xyz="0 0 0" rpy="0 0 0" />
   <geometry>
-    <mesh filename="package://racecar_description/meshes/right_rear_wheel.STL" />
+    <mesh filename="$(find maze_solver)/cartographer_config/racecar_description/meshes/right_rear_wheel.STL" />
   </geometry>
 </xacro:macro>
@@ -59,5 +59,5 @@
   <origin xyz="0 0 0" rpy="0 0 0" />
   <geometry>
-    <mesh filename="package://racecar_description/meshes/left_front_wheel.STL" />
+    <mesh filename="$(find maze_solver)/cartographer_config/racecar_description/meshes/left_front_wheel.STL" />
   </geometry>
 </xacro:macro>
@@ -65,5 +65,5 @@
   <origin xyz="0 0 0" rpy="0 0 0" />
   <geometry>
-    <mesh filename="package://racecar_description/meshes/right_front_wheel.STL" />
+    <mesh filename="$(find maze_solver)/cartographer_config/racecar_description/meshes/right_front_wheel.STL" />
   </geometry>
 </xacro:macro>
@@ -71,5 +71,5 @@
   <origin xyz="0 0 0" rpy="0 0 0" />
   <geometry>
-    <mesh filename="package://racecar_description/meshes/left_steering_hinge.STL" />
+    <mesh filename="$(find maze_solver)/cartographer_config/racecar_description/meshes/left_steering_hinge.STL" />
   </geometry>
 </xacro:macro>
@@ -77,5 +77,5 @@
   <origin xyz="0 0 0" rpy="0 0 0" />
   <geometry>
-    <mesh filename="package://racecar_description/meshes/right_steering_hinge.STL" />
+    <mesh filename="$(find maze_solver)/cartographer_config/racecar_description/meshes/right_steering_hinge.STL" />
   </geometry>
 </xacro:macro>

File: cartographer_config/racecar_description/urdf/racecar.xacro (robot description, xacro)
@@ -1,5 +1,5 @@
 <?xml version="1.0"?>
 <robot name="racecar" xmlns:xacro="http://www.ros.org/wiki/xacro">
-  <xacro:include filename="$(find racecar_description)/urdf/macros.xacro" />
+  <xacro:include filename="$(find maze_solver)/cartographer_config/racecar_description/urdf/macros.xacro" />
   <!-- Add chassis and it's inertia link -->
   <link name="base_link" />
@@ -227,5 +227,5 @@
   </joint>
   <!-- Add the remaining xacros -->
-  <xacro:include filename="$(find racecar_description)/urdf/racecar.gazebo" />
-  <xacro:include filename="$(find racecar_description)/urdf/materials.xacro" />
+  <xacro:include filename="$(find maze_solver)/cartographer_config/racecar_description/urdf/racecar.gazebo" />
+  <xacro:include filename="$(find maze_solver)/cartographer_config/racecar_description/urdf/materials.xacro" />
 </robot>
